File: interface3/pcb/pcb.kicad_sch (KiCad schematic)
At the start: 27 parts, among them J1 Conn_Coaxial, T1 Murata 78602/8JC, U1 DS34LV86T, U2 DS34LV87T, U3 Pico_W

Commit message: some pcb work
Parts:
- U3: footprint RPi_Pico:RPi_Pico_SMD_TH -> library:RPi_Pico_W_SMD_TH
Connections:
- net LED_ERROR: now also U3.10 (GPIO7); no longer U3.14 (GPIO10)
- net LED_STATUS: now also U3.11 (GPIO8); no longer U3.15 (GPIO11)
- net RX: now also U3.4 (GPIO2); no longer U3.16 (GPIO12)
- net TX_ACTIVE: now also U3.6 (GPIO4); no longer U3.5 (GPIO3)
- net TX_DELAY: now also U3.7 (GPIO5); no longer U3.6 (GPIO4)
- net ~{TX}: now also U3.5 (GPIO3); no longer U3.4 (GPIO2)
Changed lines of the file:
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@@
   (no_connect (at 123.19 71.755))
   (no_connect (at 123.19 97.155))
-  (no_connect (at 123.19 84.455))
+  (no_connect (at 123.19 107.315))
   (no_connect (at 346.71 207.01))
   (no_connect (at 158.75 86.995))
+  (no_connect (at 123.19 89.535))
   (no_connect (at 123.19 99.695))
   (no_connect (at 123.19 69.215))
@@
   (no_connect (at 289.56 180.34))
   (no_connect (at 353.06 180.34))
-  (no_connect (at 123.19 89.535))
+  (no_connect (at 123.19 102.235))
   (no_connect (at 158.75 94.615))
   (no_connect (at 158.75 114.935))
@@
   (no_connect (at 123.19 114.935))
   (no_connect (at 158.75 107.315))
-  (no_connect (at 123.19 92.075))
+  (no_connect (at 123.19 104.775))
   (no_connect (at 314.96 212.09))
   (no_connect (at 158.75 71.755))
-  (no_connect (at 123.19 94.615))
   (no_connect (at 158.75 104.775))
   (no_connect (at 158.75 102.235))
@@
     (stroke (width 0) (type default))
   )
-  (wire (pts (xy 108.585 74.295) (xy 123.19 74.295))
+  (wire (pts (xy 104.14 74.295) (xy 123.19 74.295))
     (stroke (width 0) (type default))
   )
@@
     (stroke (width 0) (type default))
   )
-  (wire (pts (xy 108.585 86.995) (xy 123.19 86.995))
+  (wire (pts (xy 104.14 86.995) (xy 123.19 86.995))
     (stroke (width 0) (type default))
   )
@@
     (stroke (width 0) (type default))
   )
-  (wire (pts (xy 121.92 107.315) (xy 123.19 107.315))
-    (stroke (width 0) (type default))
-  )
   (wire (pts (xy 289.56 217.17) (xy 289.56 209.55))
     (stroke (width 0) (type default))
@@
     (stroke (width 0) (type default))
   )
-  (wire (pts (xy 121.92 104.775) (xy 123.19 104.775))
+  (wire (pts (xy 121.92 92.075) (xy 123.19 92.075))
     (stroke (width 0) (type default))
   )
@@
     (stroke (width 0) (type default))
   )
-  (wire (pts (xy 108.585 112.395) (xy 123.19 112.395))
+  (wire (pts (xy 104.14 112.395) (xy 123.19 112.395))
     (stroke (width 0) (type default))
   )
@@
     (stroke (width 0) (type default))
   )
-  (wire (pts (xy 121.92 102.235) (xy 123.19 102.235))
+  (wire (pts (xy 121.92 94.615) (xy 123.19 94.615))
     (stroke (width 0) (type default))
   )
@@
   )
   (wire (pts (xy 302.26 107.95) (xy 304.8 107.95))
+    (stroke (width 0) (type default))
+  )
+  (wire (pts (xy 121.92 84.455) (xy 123.19 84.455))
     (stroke (width 0) (type default))
   )
@@
     (effects (font (size 2.0066 2.0066) italic) (justify left bottom))
   )
-  (global_label "RX" (shape input) (at 121.92 107.315 180)
+  (global_label "RX" (shape input) (at 121.92 76.835 180)
     (effects (font (size 1.27 1.27)) (justify right))
-    (property "Intersheetrefs" "${INTERSHEET_REFS}" (at 121.92 107.315 0)
-      (effects (font (size 1.27 1.27)) hide)
-    )
-  )
-  (global_label "TX_DELAY" (shape output) (at 121.92 81.915 180)
+    (property "Intersheetrefs" "${INTERSHEET_REFS}" (at 121.92 76.835 0)
+      (effects (font (size 1.27 1.27)) hide)
+    )
+  )
+  (global_label "TX_DELAY" (shape output) (at 121.92 84.455 180)
     (effects (font (size 1.27 1.27)) (justify right))
-    (property "Intersheetrefs" "${INTERSHEET_REFS}" (at 121.92 81.915 0)
+    (property "Intersheetrefs" "${INTERSHEET_REFS}" (at 121.92 84.455 0)
       (effects (font (size 1.27 1.27)) hide)
     )
@@
     )
   )
-  (global_label "TX_ACTIVE" (shape output) (at 121.92 79.375 180)
+  (global_label "TX_ACTIVE" (shape output) (at 121.92 81.915 180)
     (effects (font (size 1.27 1.27)) (justify right))
-    (property "Intersheetrefs" "${INTERSHEET_REFS}" (at 121.92 79.375 0)
+    (property "Intersheetrefs" "${INTERSHEET_REFS}" (at 121.92 81.915 0)
       (effects (font (size 1.27 1.27)) hide)
     )
@@
     )
   )
-  (global_label "LED_ERROR" (shape output) (at 121.92 102.235 180)
+  (global_label "LED_ERROR" (shape output) (at 121.92 92.075 180)
     (effects (font (size 1.27 1.27)) (justify right))
-    (property "Intersheetrefs" "${INTERSHEET_REFS}" (at 121.92 102.235 0)
+    (property "Intersheetrefs" "${INTERSHEET_REFS}" (at 121.92 92.075 0)
       (effects (font (size 1.27 1.27)) hide)
     )
@@
     )
   )
-  (global_label "LED_STATUS" (shape output) (at 121.92 104.775 180)
+  (global_label "LED_STATUS" (shape output) (at 121.92 94.615 180)
     (effects (font (size 1.27 1.27)) (justify right))
-    (property "Intersheetrefs" "${INTERSHEET_REFS}" (at 121.92 104.775 0)
+    (property "Intersheetrefs" "${INTERSHEET_REFS}" (at 121.92 94.615 0)
       (effects (font (size 1.27 1.27)) hide)
     )
@@
     )
   )
-  (global_label "~{TX}" (shape output) (at 121.92 76.835 180)
+  (global_label "~{TX}" (shape output) (at 121.92 79.375 180)
     (effects (font (size 1.27 1.27)) (justify right))
-    (property "Intersheetrefs" "${INTERSHEET_REFS}" (at 121.92 76.835 0)
+    (property "Intersheetrefs" "${INTERSHEET_REFS}" (at 121.92 79.375 0)
       (effects (font (size 1.27 1.27)) hide)
     )
@@
     )
   )
-  (symbol (lib_id "power:GND") (at 108.585 112.395 0) (unit 1)
+  (symbol (lib_id "power:GND") (at 104.14 112.395 0) (unit 1)
     (in_bom yes) (on_board yes) (dnp no) (fields_autoplaced)
-    (property "Reference" "#PWR04" (at 108.585 118.745 0)
-      (effects (font (size 1.27 1.27)) hide)
-    )
-    (property "Value" "GND" (at 108.585 116.84 0)
-      (effects (font (size 1.27 1.27)))
-    )
-    (property "Footprint" "" (at 108.585 112.395 0)
-      (effects (font (size 1.27 1.27)) hide)
-    )
-    (property "Datasheet" "" (at 108.585 112.395 0)
+    (property "Reference" "#PWR04" (at 104.14 118.745 0)
+      (effects (font (size 1.27 1.27)) hide)
+    )
+    (property "Value" "GND" (at 104.14 116.84 0)
+      (effects (font (size 1.27 1.27)))
+    )
+    (property "Footprint" "" (at 104.14 112.395 0)
+      (effects (font (size 1.27 1.27)) hide)
+    )
+    (property "Datasheet" "" (at 104.14 112.395 0)
       (effects (font (size 1.27 1.27)) hide)
     )
@@
     )
   )
-  (symbol (lib_id "power:GND") (at 108.585 86.995 0) (unit 1)
+  (symbol (lib_id "power:GND") (at 104.14 86.995 0) (unit 1)
     (in_bom yes) (on_board yes) (dnp no) (fields_autoplaced)
-    (property "Reference" "#PWR05" (at 108.585 93.345 0)
-      (effects (font (size 1.27 1.27)) hide)
-    )
-    (property "Value" "GND" (at 108.585 91.44 0)
-      (effects (font (size 1.27 1.27)))
-    )
-    (property "Footprint" "" (at 108.585 86.995 0)
-      (effects (font (size 1.27 1.27)) hide)
-    )
-    (property "Datasheet" "" (at 108.585 86.995 0)
+    (property "Reference" "#PWR05" (at 104.14 93.345 0)
+      (effects (font (size 1.27 1.27)) hide)
+    )
+    (property "Value" "GND" (at 104.14 91.44 0)
+      (effects (font (size 1.27 1.27)))
+    )
+    (property "Footprint" "" (at 104.14 86.995 0)
+      (effects (font (size 1.27 1.27)) hide)
+    )
+    (property "Datasheet" "" (at 104.14 86.995 0)
       (effects (font (size 1.27 1.27)) hide)
     )
@@
     )
   )
-  (symbol (lib_id "power:GND") (at 108.585 74.295 0) (unit 1)
+  (symbol (lib_id "power:GND") (at 104.14 74.295 0) (unit 1)
     (in_bom yes) (on_board yes) (dnp no) (fields_autoplaced)
-    (property "Reference" "#PWR06" (at 108.585 80.645 0)
-      (effects (font (size 1.27 1.27)) hide)
-    )
-    (property "Value" "GND" (at 108.585 78.74 0)
-      (effects (font (size 1.27 1.27)))
-    )
-    (property "Footprint" "" (at 108.585 74.295 0)
-      (effects (font (size 1.27 1.27)) hide)
-    )
-    (property "Datasheet" "" (at 108.585 74.295 0)
+    (property "Reference" "#PWR06" (at 104.14 80.645 0)
+      (effects (font (size 1.27 1.27)) hide)
+    )
+    (property "Value" "GND" (at 104.14 78.74 0)
+      (effects (font (size 1.27 1.27)))
+    )
+    (property "Footprint" "" (at 104.14 74.295 0)
+      (effects (font (size 1.27 1.27)) hide)
+    )
+    (property "Datasheet" "" (at 104.14 74.295 0)
       (effects (font (size 1.27 1.27)) hide)
     )
@@
       (effects (font (size 1.27 1.27)))
     )
-    (property "Footprint" "RPi_Pico:RPi_Pico_SMD_TH" (at 140.97 93.345 90)
-      (effects (font (size 1.27 1.27)) hide)
-    )
+    (property "Footprint" "library:RPi_Pico_W_SMD_TH" (at 140.97 93.345 90)
+      (effects (font (size 1.27 1.27)) hide)
+    )

Commit message: pcb work
Parts:
- added D5: STS, LED_SMD:LED_0603_1608Metric, symbol Device:LED
- added D6: ERR, LED_SMD:LED_0603_1608Metric, symbol Device:LED
- added R7, R9: 560, Resistor_SMD:R_0603_1608Metric_Pad0.98x0.95mm_HandSolder, symbol Device:R
- added SW1: Pico Run, Button_Switch_SMD:SW_Push_1P1T_NO_6x6mm_H9.5mm, symbol Switch:SW_Push
- C1, C2: value 0.1uF -> 0.1µ; footprint Capacitor_SMD:C_0603_1608Metric -> Capacitor_SMD:C_0603_1608Metric_Pad1.08x0.95mm_HandSolder
- C3, C4: value 0.01uF -> 0.01µ; footprint Capacitor_SMD:C_0603_1608Metric -> Capacitor_SMD:C_0603_1608Metric_Pad1.08x0.95mm_HandSolder
- D1: value GRN -> PWR
- D2: value YEL -> TX
- D3: value YEL -> RX
- D4: value RED -> NET
- R1, R2, R3, R4, R5, R6, R8: footprint Resistor_SMD:R_0603_1608Metric -> Resistor_SMD:R_0603_1608Metric_Pad0.98x0.95mm_HandSolder
- R10: renamed from R11; footprint Resistor_SMD:R_0603_1608Metric -> Resistor_SMD:R_0603_1608Metric_Pad0.98x0.95mm_HandSolder
- R11: renamed from R12; footprint Resistor_SMD:R_0603_1608Metric -> Resistor_SMD:R_0603_1608Metric_Pad0.98x0.95mm_HandSolder
- R12: renamed from R16; footprint Resistor_SMD:R_0603_1608Metric -> Resistor_SMD:R_0603_1608Metric_Pad0.98x0.95mm_HandSolder
- T1: value Murata 78602/8JC -> 78602/8JC
Connections:
- net +3V3: now also R8.1
- net GND: now also D5.1 (K), D6.1 (K), SW1.2
- net RX: no longer R11.1
- net ~{TX}: no longer R10.1
- net LED_TX: now reaches U3.26 (GPIO20)
- net LED_TX: now also R10.1
- net LED_RX: now reaches U3.27 (GPIO21)
- net LED_RX: now also R11.1
- net LED_NET: now reaches U3.29 (GPIO22)
- net LED_NET: now also R12.1
- net PICO_RUN: now reaches U3.30 (RUN)
- net PICO_RUN: now also SW1.1
- net LED_STS: now reaches U3.31 (GPIO26_ADC0)
- net LED_STS: now also R7.1
- net LED_ERR: now reaches U3.32 (GPIO27_ADC1)
- net LED_ERR: now also R9.1
- net LED_ERROR: no longer names the net of U3.10 (GPIO7)
- net LED_ERROR: no longer R12.1
- net LED_STATUS: no longer names the net of U3.11 (GPIO8)
- net LED_STATUS: no longer R8.1
- new net: D5.2 (A), R7.2
- new net: D6.2 (A), R9.2
- no-connect marks 34 -> 30

Commit message: interface3 pcb work
Parts:
- added D10: NET, LED_SMD:LED_0603_1608Metric, symbol Device:LED
- added D11: STS, LED_SMD:LED_0603_1608Metric, symbol Device:LED
- added D12: ERR, LED_SMD:LED_0603_1608Metric, symbol Device:LED
- added D7: RX3, LED_SMD:LED_0603_1608Metric, symbol Device:LED
- added D8, D9: TX3, LED_SMD:LED_0603_1608Metric, symbol Device:LED
- added J2: Conn_Coaxial, Connector_Coaxial:BNC_Amphenol_B6252HB-NPP3G-50_Horizontal, symbol Connector:Conn_Coaxial
- added J3: PMOD, Connector_PinHeader_2.54mm:PinHeader_2x06_P2.54mm_Vertical, symbol Connector_Generic:Conn_02x06_Odd_Even
- added R13, R14, R15, R16, R17, R18, R19, R20, R21, R22, R23, R24: 560, Resistor_SMD:R_0603_1608Metric_Pad0.98x0.95mm_HandSolder, symbol Device:R
- added T2: 78602/8JC, library:Murata_786J, symbol library:Murata_78602
- C2: value 0.1µ -> 0.01µ; Part EMK107B7104KA-T -> HMK107B7103KA-T
- C3: value 0.01µ -> 0.1µ; Part HMK107B7103KA-T -> EMK107B7104KA-T
- D2: value TX -> TX1
- D3: value RX -> RX1
- D4: value NET -> TX2; Part 150060RS55040 -> 150060YS55040
- D5: value STS -> RX2; Part 150060RS55040 -> 150060YS55040
- D6: value ERR -> TX3; Part 150060RS55040 -> 150060YS55040
- R1: value 150 -> 120; Part RCS0603150RFKEA -> RCS0603120RFKEA
- R10: value 560 -> 510; Part RCS0603560RFKEA -> RCS0603510RFKEA
- R11, R12: value 560 -> 33; Part RCS0603560RFKEA -> RCS060333R0FKEA
- R3: value 33 -> 150; Part RCS060333R0FKEA -> RCS0603150RFKEA
- R4: value 33 -> 510; Part RCS060333R0FKEA -> RCS0603510RFKEA
- R5: value 510 -> 33; Part RCS0603510RFKEA -> RCS060333R0FKEA
- R6: value 120 -> 33; Part RCS0603120RFKEA -> RCS060333R0FKEA
- R7: value 560 -> 120; Part RCS0603560RFKEA -> RCS0603120RFKEA
- R8, R9: value 560 -> 150; Part RCS0603560RFKEA -> RCS0603150RFKEA
Connections:
- net +3V3: now also J3.11 (Pin_11), J3.12 (Pin_12), R13.1; no longer R8.1
- net GND: now also D10.1 (K), D11.1 (K), D12.1 (K), D7.1 (K), D8.1 (K), D9.1 (K), J3.10 (Pin_10), J3.9 (Pin_9); no longer U1.1 (E-), U1.2 (E+), U2.12 (ENABLE), U2.12 (ENABLE), U2.15 (INPUT), U2.9 (INPUT)
- net LED_ERR: now also R24.1; no longer R9.1
- net LED_NET: now also R22.1; no longer R12.1
- net LED_STS: now also R23.1; no longer R7.1
- net at U2.2 (OUT+): now also R3.1; no longer R2.1
- net at U2.3 (OUT-): now also R2.2; no longer R1.2
- net at U2.5 (OUT-): now also R5.2; no longer R3.2
- net at U2.6 (OUT+): now also R6.2; no longer R4.2
- net at J1.1 (In), T1.1: now also R1.1; no longer R6.1
- net at J1.2 (Ext), T1.6: now also R1.2; no longer R6.2
- net RX2: now reaches U1.3 (OUT)
- net RX2: now also U3.12 (GPIO9)
- net at U2.10 (OUT+): now also R9.1
- net at U2.11 (OUT-): now also R8.2
- net at U2.13 (OUT-): now also R11.2
- net at U2.14 (OUT+): now also R12.2
- net at D2.2 (A): now also R14.2; no longer R10.2
- net at D3.2 (A): now also R15.2; no longer R11.2
- net at D4.2 (A): now also R16.2; no longer R12.2
- net at D1.2 (A): now also R13.2; no longer R8.2
- net at R7.2: now also J2.2 (Ext), T2.6; no longer D5.2 (A)
- net at D6.2 (A): now also R18.2; no longer R9.2
- net LED_RX1: now reaches U3.10 (GPIO7)
- net LED_RX1: now also R15.1
- net LED_TX1: now reaches U3.11 (GPIO8)
- net LED_TX1: now also R14.1
- net ~{TX2}: now reaches U3.13 (GND)
- net ~{TX2}: now also U2.15 (INPUT)
- net TX2_ACTIVE: now reaches U3.14 (GPIO10)
- net TX2_ACTIVE: now also U2.12 (ENABLE), U2.12 (ENABLE)
- net TX2_DELAY: now reaches U3.15 (GPIO11)
- net TX2_DELAY: now also U2.9 (INPUT)
- net LED_RX2: now reaches U3.16 (GPIO12)
- net LED_RX2: now also R17.1
- net LED_TX2: now reaches U3.17 (GPIO13)
- net LED_TX2: now also R16.1
- net RX3: now reaches U3.19 (GPIO14)
- net RX3: now also J3.5 (Pin_5)
- net TX3: now reaches U3.20 (GPIO15)
- net TX3: now also J3.7 (Pin_7)
- net TX3_ACTIVE: now reaches U3.21 (GPIO16)
- net TX3_ACTIVE: now also J3.1 (Pin_1)
- net TX3_DELAY: now reaches U3.22 (GPIO17)
- net TX3_DELAY: now also J3.3 (Pin_3)
- net RX4: now reaches U3.24 (GPIO18)
- net RX4: now also J3.6 (Pin_6)
- net TX4: now reaches U3.25 (GPIO19)
- net TX4: now also J3.8 (Pin_8)
- net LED_RX renamed TX2+
- net TX2+: now also R10.2, R8.1, T2.3; no longer U3.27 (GPIO21)
- net LED_TX renamed TX2-
- net TX2-: now also R12.1, R9.2, T2.4; no longer U3.26 (GPIO20)
- net RX renamed RX1
- net RX+ renamed RX1+
- net RX- renamed RX1-
- removed net TX+: R1.1, R3.1, R5.2, T1.3
- net TX- renamed TX1-
- net TX1-: now also R3.2, R6.1; no longer R2.2, R5.1
- net TX_ACTIVE renamed TX1_ACTIVE
- net TX_DELAY renamed TX1_DELAY
- net ~{TX} renamed ~{TX1}
- new net: D7.2 (A), R19.2
- new net: J2.1 (In), R7.1, T2.1
- new net: D9.2 (A), R21.2
- new net: D8.2 (A), R20.2
- new net: D5.2 (A), R17.2
- new net: D10.2 (A), R22.2
- new net: D11.2 (A), R23.2
- new net: D12.2 (A), R24.2
- new net LED_RX3: R19.1
- new net LED_TX3: R18.1, R20.1, R21.1
- new net RX2+: T2.2, U1.2 (E+)
- new net RX2-: T2.5, U1.1 (E-)
- new net TX1+: R2.1, R4.2, R5.1, T1.3
- new net TX4_ACTIVE: J3.2 (Pin_2), U3.26 (GPIO20)
- new net TX4_DELAY: J3.4 (Pin_4), U3.27 (GPIO21)
- no-connect marks 30 -> 11
Other:
- note added: "Connectors and Buttons"
- note added: "Line Drivers and Receivers"
- note removed: "Line Driver and Receiver"

Commit message: interface3 version 1 pcb sent to jlcpcb
Parts:
- added J4: POWER, Connector_USB:USB_B_OST_USB-B1HSxx_Horizontal, symbol Connector:USB_B
- D8: value TX3 -> TX4
- D9: value TX3 -> RX4
- J1: value Conn_Coaxial -> PORT1
- J2: value Conn_Coaxial -> PORT2
- J3: value PMOD -> PORT3/4
Connections:
- net GND: now also J4.4 (GND), J4.5 (Shield)
- net LED_RX3: now also U3.1 (GPIO0)
- net LED_TX3: now also U3.2 (GPIO1); no longer R20.1, R21.1
- net LED_TX4: now reaches U3.34 (GPIO28_ADC2)
- net LED_TX4: now also R20.1
- net VBUS: now reaches U3.40 (VBUS)
- net VBUS: now also J4.1 (VBUS)
- net LED_RX4: now reaches U3.9 (GPIO6)
- net LED_RX4: now also R21.1
- no-connect marks 11 -> 8
Other:
- moved on the sheet: C1, C2, C3, C4, D1, D10, D11, D12, D2, D3, D4, D5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
